Commit message: add project

File: three_wheel_robot.urdf (robot description, URDF)
Before this commit: robot ethiopia_bot, 1 links, 0 joints
Links:
- added link caster_wheel, mass 1.0; collision sphere radius=0.05; visual sphere radius=0.05
- added link left_wheel, mass 2.0; collision cylinder length=0.05 radius=0.1; visual cylinder length=0.05 radius=0.1
- added link right_wheel, mass 2.0; collision cylinder length=0.05 radius=0.1; visual cylinder length=0.05 radius=0.1
Joints:
- added joint caster_wheel_joint: type fixed, parent base_link, child caster_wheel, origin xyz=-0.15 0 -0.1
- added joint left_wheel_joint: type continuous, parent base_link, child left_wheel, origin xyz=0.1 0.17 -0.05 rpy=-1.5707 0 0, axis 0 0 1
- added joint right_wheel_joint: type continuous, parent base_link, child right_wheel, origin xyz=0.1 -0.17 -0.05 rpy=-1.5707 0 0, axis 0 0 1
